File: IV11/IV-11-breakout.kicad_pcb (KiCad board)
At the start: 2 copper layers, 25 x 62.5 mm, 8 parts, among them J1 Conn_01x12_Male, J2 LED_DOUT

Commit message: Tweaks!
Parts:
- removed R1: R, Resistor_THT:R_Axial_DIN0309_L9.0mm_D3.2mm_P12.70mm_Horizontal
- removed the REF** at (109.5, 133.6)
- added REF**: OSHW-Logo2_9.8x8mm_SilkScreen, Symbol:OSHW-Logo2_9.8x8mm_SilkScreen, B.Cu at (111.8, 129.2)
- J1: value Conn_01x12_Male -> Conn_01x13_Male; footprint Connector_PinHeader_2.54mm:PinHeader_1x12_P2.54mm_Vertical -> Connector_PinHeader_2.54mm:PinHeader_1x13_P2.54mm_Vertical
- J2: value LED_DOUT -> Conn_01x01
- moved J2 2.29 mm to (122.9, 99.7)
Connections:
- D1 pad 1: VCC -> /LED+V
- J1 pad 11: VCC -> /HEATER+V
- J1 pad 12: /LED_DIN -> /LED+V
- VFD1 pad 11: Net-(R1-Pad2) -> /HEATER+V
Routing:
- net /LED+V: track 0.00 -> 59.1 mm, vias 0 -> 2
- net /HEATER+V: track 0.00 -> 57.4 mm, vias 0 -> 2
- net VCC: track 57.0 -> 0.00 mm, vias 1 -> 0
- net Net-(R1-Pad2): track 35.6 -> 0.00 mm, vias 1 -> 0
- net /LED_DIN: track 50.7 -> 55.6 mm
- net /LED_DOUT: track 46.5 -> 48.0 mm
- net /GRID: track 52.5 -> 51.6 mm
Other:
- board size 25 x 62.5 mm -> 25 x 65 mm
- board text added: "Heat+V"
- board text added: "LED+V"
- board text added: "LED_DOUT"
- board text removed: "VCC"
