File: IV11/VFD.sch (KiCad schematic (older format))
At the start: 62 parts, among them J1 USB_B, SW1 switch, SW2 switch, SW3 switch, SW4 switch, U1 74HC595, U10 UDN2981, U11 UDN2981, U12 UDN2981, U13 WeMos_mini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

Commit message: Changes for back to front LED markings
Parts:
- D1, D2, D3, D4, D5, D6, D7, D8: symbol 5mmNeopixel:WS2812B -> 5mmNeopixel:NeoPixel_THT
- U18: symbol ChineseModules:MiniBuckBoard -> GenericModules:MP2307BuckConverterModule
- U19: symbol ChineseModules:BoostBoard -> GenericModules:MT3608BoostConverterModule
- U20: symbol ChineseModules:DS3231RTCModule -> GenericModules:DS3231RTCModule
- VFD1, VFD2, VFD3, VFD4, VFD5, VFD6, VFD7, VFD8: symbol VFD-rescue:IV-11-vfd -> vfd:IV-11
Connections:
- wire segments 592 -> 579
Changed lines of the file:
@@
 EESchema Schematic File Version 4
-LIBS:VFD-cache
 EELAYER 26 0
 EELAYER END
@@
 	4550 1250 4750 1250
 $Comp
-L VFD-rescue:IV-11-vfd VFD1
+L vfd:IV-11 VFD1
 U 1 1 5B727BC1
 P 4200 2000
@@
 	4550 3550 4750 3550
 $Comp
-L VFD-rescue:IV-11-vfd VFD3
+L vfd:IV-11 VFD3
 U 1 1 5B72D955
 P 4200 4300
@@
 	4550 5900 4750 5900
 $Comp
-L VFD-rescue:IV-11-vfd VFD5
+L vfd:IV-11 VFD5
 U 1 1 5B7320B7
 P 4200 6650
@@
 	9500 1450 9700 1450
 $Comp
-L VFD-rescue:IV-11-vfd VFD2
+L vfd:IV-11 VFD2
 U 1 1 5B73C1FB
 P 9150 2200
@@
 	9500 3750 9700 3750
 $Comp
-L VFD-rescue:IV-11-vfd VFD4
+L vfd:IV-11 VFD4
 U 1 1 5B74BC81
 P 9150 4500
@@
 	9500 5950 9700 5950
 $Comp
-L VFD-rescue:IV-11-vfd VFD6
+L vfd:IV-11 VFD6
 U 1 1 5B76357F
 P 9150 6700
@@
 	1    0    0    -1
 $EndComp
-Wire Wire Line
-	7150 9150 7150 9350
 Text GLabel 5950 9150 0    50   Input ~ 0
 SW_1
@@
 	14350 1650 14550 1650
 $Comp
-L VFD-rescue:IV-11-vfd VFD7
+L vfd:IV-11 VFD7
 U 1 1 5B4DE300
 P 14000 2400
@@
 	14350 3850 14550 3850
 $Comp
-L VFD-rescue:IV-11-vfd VFD8
+L vfd:IV-11 VFD8
 U 1 1 5B5EC07F
 P 14000 4600
@@
 $EndComp
 $Comp
-L ChineseModules:MiniBuckBoard U18
+L GenericModules:MP2307BuckConverterModule U18
 U 1 1 5B8B2710
 P 12500 8850
@@
 	13050 8350 13050 8650
 $Comp
-L ChineseModules:BoostBoard U19
+L GenericModules:MT3608BoostConverterModule U19
 U 1 1 5BAFC179
 P 14050 8750
@@
 	1000 9750 1000 10750
 $Comp
-L ChineseModules:DS3231RTCModule U20
+L GenericModules:DS3231RTCModule U20
 U 1 1 5BDC61FB
 P 4150 9700
@@
 	14000 5500 14700 5500
 $Comp
-L 5mmNeopixel:WS2812B D6
+L 5mmNeopixel:NeoPixel_THT D6
 U 1 1 5C6047BD
 P 9700 9600
@@
 $EndComp
 $Comp
-L 5mmNeopixel:WS2812B D3
+L 5mmNeopixel:NeoPixel_THT D3
 U 1 1 5C64AD7C
 P 10300 8650
@@
 $EndComp
 $Comp
-L 5mmNeopixel:WS2812B D5
+L 5mmNeopixel:NeoPixel_THT D5
 U 1 1 5C64AE2E
 P 9100 9600
@@
 $EndComp
 $Comp
-L 5mmNeopixel:WS2812B D2
+L 5mmNeopixel:NeoPixel_THT D2
 U 1 1 5C64AEE3
 P 9700 8650
@@
 $EndComp
 $Comp
-L 5mmNeopixel:WS2812B D7
+L 5mmNeopixel:NeoPixel_THT D7
 U 1 1 5C64B041
 P 10300 9600
@@
 $EndComp
 $Comp
-L 5mmNeopixel:WS2812B D8
+L 5mmNeopixel:NeoPixel_THT D8
 U 1 1 5C64B128
 P 10900 9600
@@
 $EndComp
 $Comp
-L 5mmNeopixel:WS2812B D4
+L 5mmNeopixel:NeoPixel_THT D4
 U 1 1 5C64B206
 P 10900 8650
@@
 	8600 9600 8800 9600
 Wire Wire Line
-	10900 9300 11650 9300
-Wire Wire Line
 	11650 9300 11650 8350
-Wire Wire Line
-	11650 8350 10900 8350
-Wire Wire Line
-	10900 8350 10300 8350
-Connection ~ 10900 8350
-Wire Wire Line
-	10300 8350 9700 8350
-Connection ~ 10300 8350
-Connection ~ 9700 8350
-Wire Wire Line
-	10900 8950 10300 8950
-Wire Wire Line
-	10300 8950 9700 8950
-Connection ~ 10300 8950
-Wire Wire Line
-	9700 8950 9400 8950
-Connection ~ 9700 8950
-Wire Wire Line
-	10900 9900 10300 9900
-Wire Wire Line
-	10300 9900 9700 9900
-Connection ~ 10300 9900
-Wire Wire Line
-	9700 9900 9350 9900
-Connection ~ 9700 9900
-Wire Wire Line
-	9700 9300 10300 9300
-Connection ~ 9700 9300
-Wire Wire Line
-	10300 9300 10900 9300
-Connection ~ 10300 9300
-Connection ~ 10900 9300
 $Comp
 L power:GND #PWR0184
@@
 Wire Wire Line
 	9400 8950 9100 8950
-Wire Wire Line
-	9100 9300 9700 9300
 Text GLabel 8800 8650 0    50   Input ~ 0
 LED_DATA_IN
@@
 	1    0    0    -1
 $EndComp
-Wire Wire Line
-	9400 8350 9700 8350
 $Comp
-L 5mmNeopixel:WS2812B D1
+L 5mmNeopixel:NeoPixel_THT D1
 U 1 1 5C64AC77
 P 9100 8650
@@
 	1    0    0    -1
 $EndComp
-Connection ~ 7150 9350
 Wire Wire Line
 	5950 9350 6450 9350
@@
 	7900 8550 7900 8850
 Connection ~ 7900 8850
-Wire Wire Line
-	7150 9350 7150 9850
 $Comp
 L VFD-rescue:switch-userlibs SW3
@@
 $EndComp
 Wire Wire Line
-	7150 9650 7150 9850
-Connection ~ 7150 9850
-Wire Wire Line
-	7150 9850 7150 10050
-Wire Wire Line
 	5950 9850 6700 9850
 Wire Wire Line
@@
 Wire Wire Line
 	6700 9850 6750 9850
+Wire Wire Line
+	9400 8950 10900 8950
+Wire Wire Line
+	9350 9900 10900 9900
+Wire Wire Line
+	9100 9300 11650 9300
+Wire Wire Line
+	9400 8350 11650 8350
+Wire Wire Line
+	7150 9150 7150 10050
 $EndSCHEMATC

Commit message: Fix footpring mistakes
Parts:
- SW1, SW2, SW3, SW4: symbol VFD-rescue:switch-userlibs -> Switch:SW_Push
- U10, U11, U12, U16, U17, U4, U5, U6: symbol VFD-rescue:UDN2981-userlibs -> UDN2981-THT:UDN2981-THT
Connections:
- wire segments 579 -> 584
Changed lines of the file:
@@
 EESchema Schematic File Version 4
+LIBS:VFD-cache
 EELAYER 26 0
 EELAYER END
@@
 $EndDescr
 $Comp
-L VFD-rescue:UDN2981-userlibs U4
+L UDN2981-THT:UDN2981-THT U4
 U 1 1 5B727B46
 P 3150 1800
@@
 TUBE_1_DATA_OUT
 $Comp
-L VFD-rescue:UDN2981-userlibs U5
+L UDN2981-THT:UDN2981-THT U5
 U 1 1 5B72D8DA
 P 3150 4100
@@
 TUBE_3_DATA_OUT
 $Comp
-L VFD-rescue:UDN2981-userlibs U6
+L UDN2981-THT:UDN2981-THT U6
 U 1 1 5B73203C
 P 3150 6450
@@
 TUBE_5_DATA_OUT
 $Comp
-L VFD-rescue:UDN2981-userlibs U10
+L UDN2981-THT:UDN2981-THT U10
 U 1 1 5B73C180
 P 8100 2000
@@
 TUBE_2_DATA_OUT
 $Comp
-L VFD-rescue:UDN2981-userlibs U11
+L UDN2981-THT:UDN2981-THT U11
 U 1 1 5B74BC06
 P 8100 4300
@@
 TUBE_4_DATA_OUT
 $Comp
-L VFD-rescue:UDN2981-userlibs U12
+L UDN2981-THT:UDN2981-THT U12
 U 1 1 5B763504
 P 8100 6500
@@
 F 3 "" H 6800 1050 50  0001 C CNN
 	1    6800 1050
-	1    0    0    -1
+	1    0    0    1
 $EndComp
 $Comp
@@
 F 3 "" H 1850 850 50  0001 C CNN
 	1    1850 850
-	1    0    0    -1
+	1    0    0    1
 $EndComp
 $Comp
@@
 F 3 "" H 1850 3150 50  0001 C CNN
 	1    1850 3150
-	1    0    0    -1
+	1    0    0    1
 $EndComp
 $Comp
@@
 F 3 "" H 6800 3350 50  0001 C CNN
 	1    6800 3350
-	1    0    0    -1
+	1    0    0    1
 $EndComp
 $Comp
@@
 F 3 "" H 6800 5550 50  0001 C CNN
 	1    6800 5550
-	1    0    0    -1
+	1    0    0    1
 $EndComp
 $Comp
@@
 F 3 "" H 1850 5500 50  0001 C CNN
 	1    1850 5500
-	1    0    0    -1
+	1    0    0    1
 $EndComp
 $Comp
-L VFD-rescue:switch-userlibs SW1
+L Switch:SW_Push SW1
 U 1 1 5B4854F1
 P 6950 9150
@@
 $EndComp
 $Comp
-L VFD-rescue:switch-userlibs SW2
+L Switch:SW_Push SW2
 U 1 1 5B485708
 P 6950 9350
@@
 $EndComp
 $Comp
-L VFD-rescue:UDN2981-userlibs U16
+L UDN2981-THT:UDN2981-THT U16
 U 1 1 5B4DE28E
 P 12950 2200
@@
 F 3 "" H 11650 1250 50  0001 C CNN
 	1    11650 1250
-	1    0    0    -1
+	1    0    0    1
 $EndComp
 $Comp
-L VFD-rescue:UDN2981-userlibs U17
+L UDN2981-THT:UDN2981-THT U17
 U 1 1 5B5EC00E
 P 12950 4400
@@
 F 3 "" H 11650 3450 50  0001 C CNN
 	1    11650 3450
-	1    0    0    -1
+	1    0    0    1
 $EndComp
 $Comp
@@
 Connection ~ 7900 8850
 $Comp
-L VFD-rescue:switch-userlibs SW3
+L Switch:SW_Push SW3
 U 1 1 5B83B7E0
 P 6950 9650
@@
 $EndComp
 $Comp
-L VFD-rescue:switch-userlibs SW4
+L Switch:SW_Push SW4
 U 1 1 5B83B7E7
 P 6950 9850
@@
 	6700 9850 6750 9850
 Wire Wire Line
-	9400 8950 10900 8950
+	9400 8950 10300 8950
 Wire Wire Line
-	9350 9900 10900 9900
+	9350 9900 9700 9900
 Wire Wire Line
-	9100 9300 11650 9300
+	9100 9300 9700 9300
 Wire Wire Line
-	9400 8350 11650 8350
+	9400 8350 10300 8350
 Wire Wire Line
 	7150 9150 7150 10050
+Connection ~ 10300 8950
+Wire Wire Line
+	10300 8950 10900 8950
+Connection ~ 10300 8350
+Wire Wire Line
+	10300 8350 10900 8350
+Connection ~ 10900 8350
+Wire Wire Line
+	10900 8350 11650 8350
+Connection ~ 9700 9300
+Wire Wire Line
+	9700 9300 11650 9300
+Connection ~ 9700 9900
+Wire Wire Line
+	9700 9900 10900 9900
+$Comp
+L power:+3V3 #PWR?
+U 1 1 5C6EC34C
+P 1850 850
+F 0 "#PWR?" H 1850 700 50  0001 C CNN
+F 1 "+3V3" H 1865 1023 50  0000 C CNN
+F 2 "" H 1850 850 50  0001 C CNN
+F 3 "" H 1850 850 50  0001 C CNN
+	1    1850 850
+	1    0    0    -1
+$EndComp
+$Comp
+L power:+3V3 #PWR?
+U 1 1 5C6EC466
+P 1850 3150
+F 0 "#PWR?" H 1850 3000 50  0001 C CNN
+F 1 "+3V3" H 1865 3323 50  0000 C CNN
+F 2 "" H 1850 3150 50  0001 C CNN
+F 3 "" H 1850 3150 50  0001 C CNN
+	1    1850 3150
+	1    0    0    -1
+$EndComp
+$Comp
+L power:+3V3 #PWR?
+U 1 1 5C6EC542
+P 6800 1050
+F 0 "#PWR?" H 6800 900 50  0001 C CNN
+F 1 "+3V3" H 6815 1223 50  0000 C CNN
+F 2 "" H 6800 1050 50  0001 C CNN
+F 3 "" H 6800 1050 50  0001 C CNN
+	1    6800 1050
+	1    0    0    -1
+$EndComp
+$Comp
+L power:+3V3 #PWR?
+U 1 1 5C6EC61E
+P 6800 3350
+F 0 "#PWR?" H 6800 3200 50  0001 C CNN
+F 1 "+3V3" H 6815 3523 50  0000 C CNN
+F 2 "" H 6800 3350 50  0001 C CNN
+F 3 "" H 6800 3350 50  0001 C CNN
+	1    6800 3350
+	1    0    0    -1
+$EndComp
+$Comp
+L power:+3V3 #PWR?
+U 1 1 5C6EC6FA
+P 11650 1250
+F 0 "#PWR?" H 11650 1100 50  0001 C CNN
+F 1 "+3V3" H 11665 1423 50  0000 C CNN
+F 2 "" H 11650 1250 50  0001 C CNN
+F 3 "" H 11650 1250 50  0001 C CNN
+	1    11650 1250
+	1    0    0    -1
+$EndComp
+$Comp
+L power:+3V3 #PWR?
+U 1 1 5C6EC814
+P 11650 3450
+F 0 "#PWR?" H 11650 3300 50  0001 C CNN
+F 1 "+3V3" H 11665 3623 50  0000 C CNN
+F 2 "" H 11650 3450 50  0001 C CNN
+F 3 "" H 11650 3450 50  0001 C CNN
+	1    11650 3450
+	1    0    0    -1
+$EndComp
+$Comp
+L power:+3V3 #PWR?
+U 1 1 5C6EC8F0
+P 6800 5550
+F 0 "#PWR?" H 6800 5400 50  0001 C CNN
+F 1 "+3V3" H 6815 5723 50  0000 C CNN
+F 2 "" H 6800 5550 50  0001 C CNN
+F 3 "" H 6800 5550 50  0001 C CNN
+	1    6800 5550
+	1    0    0    -1
+$EndComp
+$Comp
+L power:+3V3 #PWR?
+U 1 1 5C6ECA0A
+P 1850 5500
+F 0 "#PWR?" H 1850 5350 50  0001 C CNN
+F 1 "+3V3" H 1865 5673 50  0000 C CNN
+F 2 "" H 1850 5500 50  0001 C CNN
+F 3 "" H 1850 5500 50  0001 C CNN
+	1    1850 5500
+	1    0    0    -1
+$EndComp
 $EndSCHEMATC

Commit message: Update footprints to use the 'generic modules'
Parts:
- U18: footprint ChineseModules:BuckModule -> GenericModules:MP2307BuckConverterModule
- U19: footprint ChineseModules:MT3608BoostModule -> GenericModules:MT3608BoostConverterModule
- U20: footprint ChineseModules:DS3121RTCModule -> GenericModules:DS3121RTCModule
Changed lines of the file:
@@
 F 0 "U18" H 12550 9315 50  0000 C CNN
 F 1 "MiniBuckBoard" H 12550 9224 50  0000 C CNN
-F 2 "ChineseModules:BuckModule" H 12500 8850 50  0001 C CNN
+F 2 "GenericModules:MP2307BuckConverterModule" H 12500 8850 50  0001 C CNN
 F 3 "" H 12500 8850 50  0001 C CNN
 	1    12500 8850
@@
 F 0 "U19" H 14075 9115 50  0000 C CNN
 F 1 "BoostBoard" H 14075 9024 50  0000 C CNN
-F 2 "ChineseModules:MT3608BoostModule" H 14050 8750 50  0001 C CNN
+F 2 "GenericModules:MT3608BoostConverterModule" H 14050 8750 50  0001 C CNN
 F 3 "" H 14050 8750 50  0001 C CNN
 	1    14050 8750
@@
 F 0 "U20" H 4150 10215 50  0000 C CNN
 F 1 "DS3231RTCModule" H 4150 10124 50  0000 C CNN
-F 2 "ChineseModules:DS3121RTCModule" H 4150 9700 50  0001 C CNN
+F 2 "GenericModules:DS3121RTCModule" H 4150 9700 50  0001 C CNN
 F 3 "" H 4150 9700 50  0001 C CNN
 	1    4150 9700
@@
 	9700 9900 10900 9900
 $Comp
-L power:+3V3 #PWR?
+L power:+3V3 #PWR0199
 U 1 1 5C6EC34C
 P 1850 850
-F 0 "#PWR?" H 1850 700 50  0001 C CNN
+F 0 "#PWR0199" H 1850 700 50  0001 C CNN
 F 1 "+3V3" H 1865 1023 50  0000 C CNN
 F 2 "" H 1850 850 50  0001 C CNN
@@
 $EndComp
 $Comp
-L power:+3V3 #PWR?
+L power:+3V3 #PWR0200
 U 1 1 5C6EC466
 P 1850 3150
-F 0 "#PWR?" H 1850 3000 50  0001 C CNN
+F 0 "#PWR0200" H 1850 3000 50  0001 C CNN
 F 1 "+3V3" H 1865 3323 50  0000 C CNN
 F 2 "" H 1850 3150 50  0001 C CNN
@@
 $EndComp
 $Comp
-L power:+3V3 #PWR?
+L power:+3V3 #PWR0201
 U 1 1 5C6EC542
 P 6800 1050
-F 0 "#PWR?" H 6800 900 50  0001 C CNN
+F 0 "#PWR0201" H 6800 900 50  0001 C CNN
 F 1 "+3V3" H 6815 1223 50  0000 C CNN
 F 2 "" H 6800 1050 50  0001 C CNN
@@
 $EndComp
 $Comp
-L power:+3V3 #PWR?
+L power:+3V3 #PWR0202
 U 1 1 5C6EC61E
 P 6800 3350
-F 0 "#PWR?" H 6800 3200 50  0001 C CNN
+F 0 "#PWR0202" H 6800 3200 50  0001 C CNN
 F 1 "+3V3" H 6815 3523 50  0000 C CNN
 F 2 "" H 6800 3350 50  0001 C CNN
@@
 $EndComp
 $Comp
-L power:+3V3 #PWR?
+L power:+3V3 #PWR0203
 U 1 1 5C6EC6FA
 P 11650 1250
-F 0 "#PWR?" H 11650 1100 50  0001 C CNN
+F 0 "#PWR0203" H 11650 1100 50  0001 C CNN
 F 1 "+3V3" H 11665 1423 50  0000 C CNN
 F 2 "" H 11650 1250 50  0001 C CNN
@@
 $EndComp
 $Comp
-L power:+3V3 #PWR?
+L power:+3V3 #PWR0204
 U 1 1 5C6EC814
 P 11650 3450
-F 0 "#PWR?" H 11650 3300 50  0001 C CNN
+F 0 "#PWR0204" H 11650 3300 50  0001 C CNN
 F 1 "+3V3" H 11665 3623 50  0000 C CNN
 F 2 "" H 11650 3450 50  0001 C CNN
@@
 $EndComp
 $Comp
-L power:+3V3 #PWR?
+L power:+3V3 #PWR0205
 U 1 1 5C6EC8F0
 P 6800 5550
-F 0 "#PWR?" H 6800 5400 50  0001 C CNN
+F 0 "#PWR0205" H 6800 5400 50  0001 C CNN
 F 1 "+3V3" H 6815 5723 50  0000 C CNN
 F 2 "" H 6800 5550 50  0001 C CNN
@@
 $EndComp
 $Comp
-L power:+3V3 #PWR?
+L power:+3V3 #PWR0206
 U 1 1 5C6ECA0A
 P 1850 5500
-F 0 "#PWR?" H 1850 5350 50  0001 C CNN
+F 0 "#PWR0206" H 1850 5350 50  0001 C CNN
 F 1 "+3V3" H 1865 5673 50  0000 C CNN
 F 2 "" H 1850 5500 50  0001 C CNN

Commit message: Finish import of new neopixel footprint and associated groundfill changes
Connections:
- wire segments 584 -> 598
Other:
- moved on the sheet: D9
Changed lines of the file:
@@
 L 5mmNeopixel:NeoPixel_THT D6
 U 1 1 5C6047BD
-P 9700 9600
-F 0 "D6" H 10041 9646 50  0000 L CNN
-F 1 "WS2812B" H 10041 9555 50  0000 L CNN
-F 2 "LED_THT:LED_D5.0mm-4" H 9750 9300 50  0001 L TNN
-F 3 "https://cdn-shop.adafruit.com/datasheets/WS2812B.pdf" H 9800 9225 50  0001 L TNN
-	1    9700 9600
+P 9750 9600
+F 0 "D6" H 10091 9646 50  0000 L CNN
+F 1 "WS2812B" H 10091 9555 50  0000 L CNN
+F 2 "LED_THT:LED_D5.0mm-4" H 9800 9300 50  0001 L TNN
+F 3 "https://cdn-shop.adafruit.com/datasheets/WS2812B.pdf" H 9850 9225 50  0001 L TNN
+	1    9750 9600
 	1    0    0    -1
 $EndComp
@@
 L 5mmNeopixel:NeoPixel_THT D3
 U 1 1 5C64AD7C
-P 10300 8650
-F 0 "D3" H 10641 8696 50  0000 L CNN
-F 1 "WS2812B" H 10641 8605 50  0000 L CNN
-F 2 "LED_THT:LED_D5.0mm-4" H 10350 8350 50  0001 L TNN
-F 3 "https://cdn-shop.adafruit.com/datasheets/WS2812B.pdf" H 10400 8275 50  0001 L TNN
-	1    10300 8650
+P 10400 8650
+F 0 "D3" H 10741 8696 50  0000 L CNN
+F 1 "WS2812B" H 10741 8605 50  0000 L CNN
+F 2 "LED_THT:LED_D5.0mm-4" H 10450 8350 50  0001 L TNN
+F 3 "https://cdn-shop.adafruit.com/datasheets/WS2812B.pdf" H 10500 8275 50  0001 L TNN
+	1    10400 8650
 	1    0    0    -1
 $EndComp
@@
 L 5mmNeopixel:NeoPixel_THT D2
 U 1 1 5C64AEE3
-P 9700 8650
-F 0 "D2" H 10041 8696 50  0000 L CNN
-F 1 "WS2812B" H 10041 8605 50  0000 L CNN
-F 2 "LED_THT:LED_D5.0mm-4" H 9750 8350 50  0001 L TNN
-F 3 "https://cdn-shop.adafruit.com/datasheets/WS2812B.pdf" H 9800 8275 50  0001 L TNN
-	1    9700 8650
+P 9750 8650
+F 0 "D2" H 10091 8696 50  0000 L CNN
+F 1 "WS2812B" H 10091 8605 50  0000 L CNN
+F 2 "LED_THT:LED_D5.0mm-4" H 9800 8350 50  0001 L TNN
+F 3 "https://cdn-shop.adafruit.com/datasheets/WS2812B.pdf" H 9850 8275 50  0001 L TNN
+	1    9750 8650
 	1    0    0    -1
 $EndComp
@@
 L 5mmNeopixel:NeoPixel_THT D7
 U 1 1 5C64B041
-P 10300 9600
-F 0 "D7" H 10641 9646 50  0000 L CNN
-F 1 "WS2812B" H 10641 9555 50  0000 L CNN
-F 2 "LED_THT:LED_D5.0mm-4" H 10350 9300 50  0001 L TNN
-F 3 "https://cdn-shop.adafruit.com/datasheets/WS2812B.pdf" H 10400 9225 50  0001 L TNN
-	1    10300 9600
+P 10400 9600
+F 0 "D7" H 10741 9646 50  0000 L CNN
+F 1 "WS2812B" H 10741 9555 50  0000 L CNN
+F 2 "LED_THT:LED_D5.0mm-4" H 10450 9300 50  0001 L TNN
+F 3 "https://cdn-shop.adafruit.com/datasheets/WS2812B.pdf" H 10500 9225 50  0001 L TNN
+	1    10400 9600
 	1    0    0    -1
 $EndComp
@@
 L 5mmNeopixel:NeoPixel_THT D8
 U 1 1 5C64B128
-P 10900 9600
-F 0 "D8" H 11241 9646 50  0000 L CNN
-F 1 "WS2812B" H 11241 9555 50  0000 L CNN
-F 2 "LED_THT:LED_D5.0mm-4" H 10950 9300 50  0001 L TNN
-F 3 "https://cdn-shop.adafruit.com/datasheets/WS2812B.pdf" H 11000 9225 50  0001 L TNN
-	1    10900 9600
+P 11050 9600
+F 0 "D8" H 11391 9646 50  0000 L CNN
+F 1 "WS2812B" H 11391 9555 50  0000 L CNN
+F 2 "LED_THT:LED_D5.0mm-4" H 11100 9300 50  0001 L TNN
+F 3 "https://cdn-shop.adafruit.com/datasheets/WS2812B.pdf" H 11150 9225 50  0001 L TNN
+	1    11050 9600
 	1    0    0    -1
 $EndComp
@@
 L 5mmNeopixel:NeoPixel_THT D4
 U 1 1 5C64B206
-P 10900 8650
-F 0 "D4" H 11241 8696 50  0000 L CNN
-F 1 "WS2812B" H 11241 8605 50  0000 L CNN
-F 2 "LED_THT:LED_D5.0mm-4" H 10950 8350 50  0001 L TNN
-F 3 "https://cdn-shop.adafruit.com/datasheets/WS2812B.pdf" H 11000 8275 50  0001 L TNN
-	1    10900 8650
-	1    0    0    -1
-$EndComp
-Wire Wire Line
-	11200 8650 11200 9200
-Wire Wire Line
-	11200 9200 8600 9200
+P 11100 8650
+F 0 "D4" H 11441 8696 50  0000 L CNN
+F 1 "WS2812B" H 11441 8605 50  0000 L CNN
+F 2 "LED_THT:LED_D5.0mm-4" H 11150 8350 50  0001 L TNN
+F 3 "https://cdn-shop.adafruit.com/datasheets/WS2812B.pdf" H 11200 8275 50  0001 L TNN
+	1    11100 8650
+	1    0    0    -1
+$EndComp
 Wire Wire Line
 	8600 9200 8600 9600
@@
 L power:GND #PWR0185
 U 1 1 5CA9AD57
-P 9400 8950
-F 0 "#PWR0185" H 9400 8700 50  0001 C CNN
-F 1 "GND" H 9405 8777 50  0000 C CNN
-F 2 "" H 9400 8950 50  0001 C CNN
-F 3 "" H 9400 8950 50  0001 C CNN
-	1    9400 8950
-	1    0    0    -1
-$EndComp
-Connection ~ 9400 8950
-Wire Wire Line
-	9400 8950 9100 8950
-Text GLabel 8800 8650 0    50   Input ~ 0
+P 9450 8950
+F 0 "#PWR0185" H 9450 8700 50  0001 C CNN
+F 1 "GND" H 9455 8777 50  0000 C CNN
+F 2 "" H 9450 8950 50  0001 C CNN
+F 3 "" H 9450 8950 50  0001 C CNN
+	1    9450 8950
+	1    0    0    -1
+$EndComp
+Text GLabel 8750 8650 0    50   Input ~ 0
 LED_DATA_IN
-Text GLabel 11200 9600 2    50   Input ~ 0
+Text GLabel 11400 9600 2    50   Input ~ 0
 LED_DATA_OUT
 $Comp
 L power:+5V #PWR0186
 U 1 1 5B5A732B
-P 9400 8350
-F 0 "#PWR0186" H 9400 8200 50  0001 C CNN
-F 1 "+5V" H 9415 8523 50  0000 C CNN
-F 2 "" H 9400 8350 50  0001 C CNN
-F 3 "" H 9400 8350 50  0001 C CNN
-	1    9400 8350
-	1    0    0    -1
-$EndComp
-$Comp
-L 5mmNeopixel:NeoPixel_THT D1
-U 1 1 5C64AC77
-P 9100 8650
-F 0 "D1" H 9441 8696 50  0000 L CNN
-F 1 "WS2812B" H 9441 8605 50  0000 L CNN
-F 2 "LED_THT:LED_D5.0mm-4" H 9150 8350 50  0001 L TNN
-F 3 "https://cdn-shop.adafruit.com/datasheets/WS2812B.pdf" H 9200 8275 50  0001 L TNN
-	1    9100 8650
+P 9450 8350
+F 0 "#PWR0186" H 9450 8200 50  0001 C CNN
+F 1 "+5V" H 9465 8523 50  0000 C CNN
+F 2 "" H 9450 8350 50  0001 C CNN
+F 3 "" H 9450 8350 50  0001 C CNN
+	1    9450 8350
 	1    0    0    -1
 $EndComp
@@
 L Device:D D9
 U 1 1 5B5A7599
-P 9250 8350
-F 0 "D9" H 9250 8566 50  0000 C CNN
-F 1 "D" H 9250 8475 50  0000 C CNN
-F 2 "Diode_THT:D_DO-35_SOD27_P7.62mm_Horizontal" H 9250 8350 50  0001 C CNN
-F 3 "~" H 9250 8350 50  0001 C CNN
-	1    9250 8350
-	1    0    0    -1
-$EndComp
-Connection ~ 9400 8350
+P 9300 8350
+F 0 "D9" H 9300 8566 50  0000 C CNN
+F 1 "D" H 9300 8475 50  0000 C CNN
+F 2 "Diode_THT:D_DO-35_SOD27_P7.62mm_Horizontal" H 9300 8350 50  0001 C CNN
+F 3 "~" H 9300 8350 50  0001 C CNN
+	1    9300 8350
+	1    0    0    -1
+$EndComp
+Connection ~ 9450 8350
 $Comp
 L power:+3V3 #PWR0146
@@
 	6700 9850 6750 9850
 Wire Wire Line
-	9400 8950 10300 8950
-Wire Wire Line
-	9350 9900 9700 9900
-Wire Wire Line
-	9100 9300 9700 9300
-Wire Wire Line
-	9400 8350 10300 8350
+	9450 8950 9750 8950
+Wire Wire Line
+	9450 8350 9750 8350
 Wire Wire Line
 	7150 9150 7150 10050
-Connection ~ 10300 8950
-Wire Wire Line
-	10300 8950 10900 8950
-Connection ~ 10300 8350
-Wire Wire Line
-	10300 8350 10900 8350
-Connection ~ 10900 8350
-Wire Wire Line
-	10900 8350 11650 8350
-Connection ~ 9700 9300
-Wire Wire Line
-	9700 9300 11650 9300
-Connection ~ 9700 9900
-Wire Wire Line
-	9700 9900 10900 9900
+Wire Wire Line
+	10400 8950 11100 8950
 $Comp
 L power:+3V3 #PWR0199
@@
 	1    0    0    -1
 $EndComp
+Wire Wire Line
+	11100 8350 11650 8350
+Connection ~ 11100 8350
+Wire Wire Line
+	10400 8350 11100 8350
+Connection ~ 9750 8350
+Connection ~ 9750 8950
+Connection ~ 10400 8350
+Connection ~ 10400 8950
+Wire Wire Line
+	9750 8350 10400 8350
+Wire Wire Line
+	9750 8950 10400 8950
+$Comp
+L 5mmNeopixel:NeoPixel_THT D1
+U 1 1 5C64AC77
+P 9100 8650
+F 0 "D1" H 9441 8696 50  0000 L CNN
+F 1 "WS2812B" H 9441 8605 50  0000 L CNN
+F 2 "LED_THT:LED_D5.0mm-4" H 9150 8350 50  0001 L TNN
+F 3 "https://cdn-shop.adafruit.com/datasheets/WS2812B.pdf" H 9200 8275 50  0001 L TNN
+	1    9100 8650
+	1    0    0    -1
+$EndComp
+Connection ~ 9750 9300
+Connection ~ 9750 9900
+Wire Wire Line
+	10400 9900 11050 9900
+Wire Wire Line
+	11050 9300 11650 9300
+Wire Wire Line
+	9350 9900 9750 9900
+Wire Wire Line
+	9100 9300 9750 9300
+Connection ~ 10400 9300
+Connection ~ 10400 9900
+Wire Wire Line
+	9750 9300 10400 9300
+Wire Wire Line
+	9750 9900 10400 9900
+Connection ~ 11050 9300
+Wire Wire Line
+	10400 9300 11050 9300
+Wire Wire Line
+	9150 8350 9100 8350
+Wire Wire Line
+	9450 8950 9100 8950
+Connection ~ 9450 8950
+Wire Wire Line
+	9400 8650 9450 8650
+Wire Wire Line
+	10050 8650 10100 8650
+Wire Wire Line
+	10700 8650 10800 8650
+Wire Wire Line
+	11400 8650 11400 9200
+Wire Wire Line
+	8600 9200 11400 9200
+Wire Wire Line
+	11350 9600 11400 9600
+Wire Wire Line
+	10750 9600 10700 9600
+Wire Wire Line
+	10100 9600 10050 9600
+Wire Wire Line
+	9450 9600 9400 9600
+Wire Wire Line
+	8750 8650 8800 8650
 $EndSCHEMATC
