File: IV11/VFD.sch (KiCad schematic (older format))
At the start: 62 parts, among them J1 USB_B, SW1 switch, SW2 switch, SW3 switch, SW4 switch, U1 74HC595, U10 UDN2981, U11 UDN2981, U12 UDN2981, U13 WeMos_mini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

Commit message: Updates to use further-spaced LED footprints for the 5mm neopixels to make rework easier!
Parts:
- D1, D2, D3, D4, D5, D6, D7, D8: footprint LED_THT:LED_D5.0mm-4 -> 5mm-neopixel-wide:LED_D5.0mm-4-Wide
Changed lines of the file:
@@
 F 0 "D6" H 10091 9646 50  0000 L CNN
 F 1 "WS2812B" H 10091 9555 50  0000 L CNN
-F 2 "LED_THT:LED_D5.0mm-4" H 9800 9300 50  0001 L TNN
+F 2 "5mm-neopixel-wide:LED_D5.0mm-4-Wide" H 9800 9300 50  0001 L TNN
 F 3 "https://cdn-shop.adafruit.com/datasheets/WS2812B.pdf" H 9850 9225 50  0001 L TNN
 	1    9750 9600
@@
 F 0 "D3" H 10741 8696 50  0000 L CNN
 F 1 "WS2812B" H 10741 8605 50  0000 L CNN
-F 2 "LED_THT:LED_D5.0mm-4" H 10450 8350 50  0001 L TNN
+F 2 "5mm-neopixel-wide:LED_D5.0mm-4-Wide" H 10450 8350 50  0001 L TNN
 F 3 "https://cdn-shop.adafruit.com/datasheets/WS2812B.pdf" H 10500 8275 50  0001 L TNN
 	1    10400 8650
@@
 F 0 "D5" H 9441 9646 50  0000 L CNN
 F 1 "WS2812B" H 9441 9555 50  0000 L CNN
-F 2 "LED_THT:LED_D5.0mm-4" H 9150 9300 50  0001 L TNN
+F 2 "5mm-neopixel-wide:LED_D5.0mm-4-Wide" H 9150 9300 50  0001 L TNN
 F 3 "https://cdn-shop.adafruit.com/datasheets/WS2812B.pdf" H 9200 9225 50  0001 L TNN
 	1    9100 9600
@@
 F 0 "D2" H 10091 8696 50  0000 L CNN
 F 1 "WS2812B" H 10091 8605 50  0000 L CNN
-F 2 "LED_THT:LED_D5.0mm-4" H 9800 8350 50  0001 L TNN
+F 2 "5mm-neopixel-wide:LED_D5.0mm-4-Wide" H 9800 8350 50  0001 L TNN
 F 3 "https://cdn-shop.adafruit.com/datasheets/WS2812B.pdf" H 9850 8275 50  0001 L TNN
 	1    9750 8650
@@
 F 0 "D7" H 10741 9646 50  0000 L CNN
 F 1 "WS2812B" H 10741 9555 50  0000 L CNN
-F 2 "LED_THT:LED_D5.0mm-4" H 10450 9300 50  0001 L TNN
+F 2 "5mm-neopixel-wide:LED_D5.0mm-4-Wide" H 10450 9300 50  0001 L TNN
 F 3 "https://cdn-shop.adafruit.com/datasheets/WS2812B.pdf" H 10500 9225 50  0001 L TNN
 	1    10400 9600
@@
 F 0 "D8" H 11391 9646 50  0000 L CNN
 F 1 "WS2812B" H 11391 9555 50  0000 L CNN
-F 2 "LED_THT:LED_D5.0mm-4" H 11100 9300 50  0001 L TNN
+F 2 "5mm-neopixel-wide:LED_D5.0mm-4-Wide" H 11100 9300 50  0001 L TNN
 F 3 "https://cdn-shop.adafruit.com/datasheets/WS2812B.pdf" H 11150 9225 50  0001 L TNN
 	1    11050 9600
@@
 F 0 "D4" H 11441 8696 50  0000 L CNN
 F 1 "WS2812B" H 11441 8605 50  0000 L CNN
-F 2 "LED_THT:LED_D5.0mm-4" H 11150 8350 50  0001 L TNN
+F 2 "5mm-neopixel-wide:LED_D5.0mm-4-Wide" H 11150 8350 50  0001 L TNN
 F 3 "https://cdn-shop.adafruit.com/datasheets/WS2812B.pdf" H 11200 8275 50  0001 L TNN
 	1    11100 8650
@@
 F 0 "D1" H 9441 8696 50  0000 L CNN
 F 1 "WS2812B" H 9441 8605 50  0000 L CNN
-F 2 "LED_THT:LED_D5.0mm-4" H 9150 8350 50  0001 L TNN
+F 2 "5mm-neopixel-wide:LED_D5.0mm-4-Wide" H 9150 8350 50  0001 L TNN
 F 3 "https://cdn-shop.adafruit.com/datasheets/WS2812B.pdf" H 9200 8275 50  0001 L TNN
 	1    9100 8650

Commit message: Fixes for not using D0 for the LEDs...
Parts:
- R5: value 10k -> 100k
Connections:
- wire segments 598 -> 597
Changed lines of the file:
@@
 L power:GND #PWR0157
 U 1 1 5C2BC43E
-P 7850 9900
-F 0 "#PWR0157" H 7850 9650 50  0001 C CNN
-F 1 "GND" H 7855 9727 50  0000 C CNN
-F 2 "" H 7850 9900 50  0001 C CNN
-F 3 "" H 7850 9900 50  0001 C CNN
-	1    7850 9900
-	1    0    0    -1
-$EndComp
-Wire Wire Line
-	7900 9350 7900 9900
-Wire Wire Line
-	7900 9900 7850 9900
+P 7900 9950
+F 0 "#PWR0157" H 7900 9700 50  0001 C CNN
+F 1 "GND" H 7905 9777 50  0000 C CNN
+F 2 "" H 7900 9950 50  0001 C CNN
+F 3 "" H 7900 9950 50  0001 C CNN
+	1    7900 9950
+	1    0    0    -1
+$EndComp
 Text GLabel 2300 10250 2    50   Input ~ 0
 LDR_IN
@@
 Text GLabel 2300 9850 2    50   Input ~ 0
 SHIFT_OE
+Text GLabel 2300 9950 2    50   Input ~ 0
+LED_DATA_IN
 Text GLabel 2300 10150 2    50   Input ~ 0
-LED_DATA_IN
-Text GLabel 2300 9950 2    50   Input ~ 0
 SW_1
 Text GLabel 2300 10050 2    50   Input ~ 0
@@
 P 7350 8400
 F 0 "R5" H 7420 8446 50  0000 L CNN
-F 1 "10k" H 7420 8355 50  0000 L CNN
+F 1 "100k" H 7420 8355 50  0000 L CNN
 F 2 "Resistor_THT:R_Axial_DIN0411_L9.9mm_D3.6mm_P12.70mm_Horizontal" V 7280 8400 50  0001 C CNN
 F 3 "~" H 7350 8400 50  0001 C CNN
@@
 Wire Wire Line
 	8750 8650 8800 8650
+Wire Wire Line
+	7900 9350 7900 9950
 $EndSCHEMATC

Commit message: V1.1 board completed, + gerbers
Parts:
- added U21: DS18B20, Connector_PinHeader_2.54mm:PinHeader_1x03_P2.54mm_Vertical, symbol Sensor_Temperature:DS18B20
Other:
- note added: "Optional DS18B20\ninstead of SW1"
Changed lines of the file:
@@
 	8700 3850 8650 3850
-Wire Wire Line
-	8650 3850 8650 4000
 Wire Wire Line
 	8650 4000 8500 4000
@@
 Wire Wire Line
 	8700 6050 8650 6050
-Wire Wire Line
-	8650 6050 8650 6200
 Wire Wire Line
 	8650 6200 8500 6200
@@
 Wire Wire Line
 	7900 9350 7900 9950
+$Comp
+L Sensor_Temperature:DS18B20 U21
+U 1 1 5B70AEE5
+P 11250 6100
+F 0 "U21" H 11020 6146 50  0000 R CNN
+F 1 "DS18B20" H 11020 6055 50  0000 R CNN
+F 2 "Connector_PinHeader_2.54mm:PinHeader_1x03_P2.54mm_Vertical" H 10250 5850 50  0001 C CNN
+F 3 "http://datasheets.maximintegrated.com/en/ds/DS18B20.pdf" H 11100 6350 50  0001 C CNN
+	1    11250 6100
+	1    0    0    -1
+$EndComp
+Wire Wire Line
+	8650 6050 8650 6200
+Wire Wire Line
+	8650 3850 8650 4000
+$Comp
+L power:GND #PWR0207
+U 1 1 5B7663A8
+P 11250 6400
+F 0 "#PWR0207" H 11250 6150 50  0001 C CNN
+F 1 "GND" H 11255 6227 50  0000 C CNN
+F 2 "" H 11250 6400 50  0001 C CNN
+F 3 "" H 11250 6400 50  0001 C CNN
+	1    11250 6400
+	1    0    0    -1
+$EndComp
+$Comp
+L power:+3V3 #PWR0208
+U 1 1 5B76650C
+P 11250 5800
+F 0 "#PWR0208" H 11250 5650 50  0001 C CNN
+F 1 "+3V3" H 11265 5973 50  0000 C CNN
+F 2 "" H 11250 5800 50  0001 C CNN
+F 3 "" H 11250 5800 50  0001 C CNN
+	1    11250 5800
+	1    0    0    -1
+$EndComp
+Text GLabel 11550 6100 2    50   Input ~ 0
+SW_1
+Text Notes 12000 5850 2    50   ~ 0
+Optional DS18B20\ninstead of SW1
 $EndSCHEMATC

Commit message: Fix bug for switches not being connected to ground!
Connections:
- wire segments 597 -> 600
Changed lines of the file:
@@
 	9450 8350 9750 8350
-Wire Wire Line
-	7150 9150 7150 10050
 Wire Wire Line
 	10400 8950 11100 8950
@@
 Text Notes 12000 5850 2    50   ~ 0
 Optional DS18B20\ninstead of SW1
+Wire Wire Line
+	7150 9150 7150 9350
+Wire Wire Line
+	7150 9350 7150 9650
+Connection ~ 7150 9350
+Wire Wire Line
+	7150 9650 7150 9850
+Connection ~ 7150 9650
+Wire Wire Line
+	7150 9850 7150 10050
+Connection ~ 7150 9850
 $EndSCHEMATC
